File: hardware/RB3200-ESP32universal.sch (EAGLE design)
At the start: 103 parts, among them IC1 FT232R, IC2 7805, T1 BC337, T2 BC337, U1 ESP-WROOM-32, U2 UM18533, X1 USB-MICRO-B-BOTTOM

Commit message: Add information text about license and authors
Other:
- note added: "Released under the Creative Commons Attribution-ShareAlike 4.0 License https://creativecommons.org/licenses/by-sa/4.0/ Designed by: JM & JP & JS & JV & RobotikaBrno RB3200-ESP32universal https://github.com/RoboticsBrno/RB3200-ESP32universal RobotikaBrno.cz Robotarna"
- note added: "RobotikaBrno"
- note added: "github:roboticsbrno/ RB3200-ESP32universal RobotikaBrno.cz Robotarna CC BY-SA 4.0"
- note removed: "ESP32 universal board Robotarna github:roboticsbrno/ RB3200-ESP32universal CC BY-SA 4.0"
- note removed: "RobotikaBrno.cz"
Changed lines of the file:
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@@
 <sheet>
 <plain>
-<text x="289.56" y="5.08" size="2.54" layer="97">ESP32 universal board
+<text x="289.306" y="4.572" size="2.1844" layer="97" font="vector">github:roboticsbrno/
+RB3200-ESP32universal
+RobotikaBrno.cz
 Robotarna
-github:roboticsbrno/
-RB3200-ESP32universal
 CC BY-SA 4.0</text>
-<text x="344.17" y="20.32" size="2.54" layer="97" ratio="14">RobotikaBrno.cz</text>
-<text x="375.92" y="5.08" size="2.54" layer="97" ratio="14">v1.0</text>
+<text x="344.17" y="20.32" size="2.54" layer="97" font="vector" ratio="14">RobotikaBrno</text>
+<text x="374.65" y="5.08" size="2.54" layer="97" font="vector" ratio="14">v1.0</text>
 <rectangle x1="338.570040625" y1="18.3900375" x2="338.783396875" y2="18.4002" layer="102"/>
 <rectangle x1="338.4278" y1="18.4002" x2="338.9256375" y2="18.41035625" layer="102"/>
@@
 <rectangle x1="338.214440625" y1="23.1652375" x2="339.138996875" y2="23.1754" layer="102"/>
 <rectangle x1="338.2754" y1="23.1754" x2="339.0882" y2="23.18555625" layer="102"/>
+<text x="180.34" y="20.32" size="1.778" layer="97" font="vector" align="center">Released under the Creative Commons Attribution-ShareAlike 4.0 License
+https://creativecommons.org/licenses/by-sa/4.0/
+Designed by: JM &amp; JP &amp; JS &amp; JV &amp; RobotikaBrno
+RB3200-ESP32universal
+https://github.com/RoboticsBrno/RB3200-ESP32universal
+RobotikaBrno.cz
+Robotarna</text>
 </plain>
 <instances>

Commit message: Publish version 2.0 of RB3200-ESP32universal and level_shifter DPS
Parts:
- removed C12: 4u7, rcl_upravena:C-EUC0805
- removed C13: 100n, rcl_upravena:C-EUC0402
- removed C14: 22u/16V, rcl_upravena:CPOL-EUSMCB
- removed D3: skl34, diode:SHOTTKY-SOD123
- removed IC1: FT232R, ftdichip_upravena:FT232R
- removed JP10, JP9: (no value), pinhead:PINHD-2X4
- removed JP12: (no value), pinhead:PINHD-1X12
- removed JP13: (no value), pinhead:PINHD-1X8
- removed JP16, JP17, JP18, JP19, JP20, JP21, LED0: (no value), pinhead:PINHD-1X1
- removed LED0-N, LED0-P, LED1-N, LED1-P, LED2-N, LED2-P, LED3-N, LED3-P: green, led:LEDCHIPLED_0603
- removed LED_CBUS2, LED_CBUS3, LED_CBUS4: yellow, led:LEDCHIP-LED0603
- added !CTS, !DCD, !DSR, !DTR, !RESET, !RTS, !SUSPEND, CHR0, CHR1, CHREN, IO0/TXLED, IO1/RXLED, IO2/RS485, IO3/WAKEUP, IO4, IO5, IO6, RI/CLK, RXD, SUSPEND, TXD: PINH1X01, pinhead_smd:PINH1X01
- added +5V, SERVOS: (no value), pinhead:PINHD-2X6
- added B1, B2: TACTM-35N-F, TACTM-35N-F:TACTM-35N-F
- added C20, C21: 100n/16V, rcl_upravena:C-EUC0402
- added C37: 330u/16V, rcl_upravena:CPOL-EUE5-10.5
- added C67, C70: 4u7/16V, rcl_upravena:C-EUC0805
- added D5: skl34, diode:SHOTTKY-SOD123
- added EN, JP36, JP38, VUSB: (no value), pinhead:PINHD-1X2
- added IC3: CP2102N-28, CP2102N:CP2102N-28
- added LED0N, LED1N, LED2N, LED3N, LED4N, LED5N: red, led:LEDCHIPLED_0603
- added LED0P, LED1P, LED2P, LED3P, LED4P, LED5P, LED_3V3_USB: green, led:LEDCHIPLED_0603
- added LEDS, VCC, VCCIO: (no value), pinhead:PINHD-2X3
- added NC28: NC, NC:NC
- added R35, R50, R51: 10k, rcl_upravena:R-EU_R0603
- added R36, R46, R48: 470R, rcl_upravena:R-EU_R0603
- added R37: 100k, rcl_upravena:R-EU_R0603
- added R47, R49: 680R, rcl_upravena:R-EU_R0603
- added U3: ARDUINOR3-BPLACE, adafruit:ARDUINOR3-BPLACE
- added USB: (no value), pinhead:PINHD-1X5
- C1, C6, C7: value 100n -> 100n/16V
- C10, C3, C5, C9: value 4u7 -> 4u7/16V
- C11: value 4u7 -> 100n/16V; device rcl_upravena:C-EUC0805 -> rcl_upravena:C-EUC0402
- C2, C4: value 100n -> 4u7/16V; device rcl_upravena:C-EUC0402 -> rcl_upravena:C-EUC0603
- C8: value 22u/16V -> 4u7/16V; device rcl_upravena:CPOL-EUSMCB -> rcl_upravena:C-EUC0805
- D1: value (none) -> skl34; device diode:DIODE-MINIMELF -> diode:SHOTTKY-SOD123
- JP11: device pinhead:PINHD-1X14 -> pinhead:PINHD-1X8
- LED1, LED2, LED3: value (none) -> yellow; device pinhead:PINHD-1X1 -> led:LEDCHIP-LED0603
- R1, R2, R26, R3, R38, R40, R42, R44: value 180R -> 470R
- R39, R41, R43, R45: value 180R -> 680R
Connections:
- net LED renamed LED_3V3
- removed net !CTS: IC1.!CTS, JP17.1
- removed net !DCD: IC1.!DCD, JP19.1
- removed net !DSR: IC1.!DSR, JP18.1
- removed net !RI: IC1.!RI, JP20.1
- removed net 3V3_FTDI: C2.1, IC1.3V3OUT
- removed net 5V->3V3: C14.+, C4.1, D2.C, U2.!SHDN, U2.IN
- removed net CBUS0: IC1.CBUS0, JP16.1
- removed net CBUS1: IC1.CBUS1, JP21.1
- removed net CBUS2: IC1.CBUS2, R1.2
- removed net CBUS2_LED: LED_CBUS2.C, R1.1
- removed net CBUS3: IC1.CBUS3, R2.2
- removed net CBUS3_LED: LED_CBUS3.C, R2.1
- removed net CBUS4: IC1.CBUS4, R3.2
- removed net CBUS4_LED: LED_CBUS4.C, R3.1
- removed net LED0: LED0.1, R38.1, R39.1
- removed net LED0-N: LED0-N.C, R39.2
- removed net LED0-P: LED0-P.A, R38.2
- removed net LED1: LED1.1, R40.1, R41.1
- removed net LED1-N: LED1-N.C, R41.2
- removed net LED1-P: LED1-P.A, R40.2
- removed net LED2: LED2.1, R42.1, R43.1
- removed net LED2-N: LED2-N.C, R43.2
- removed net LED2-P: LED2-P.A, R42.2
- removed net LED3-N: LED3-N.C, R45.2
- removed net LED3-P: LED3-P.A, R44.2
- removed net N$10: JP2.5, JP2.6, JP3.6, R7.1
- removed net N$11: JP2.3, JP2.4, JP3.4, R6.1
- removed net N$12: JP2.1, JP2.2, JP3.2, R19.1
- removed net N$13: JP6.25, JP6.26, JP7.25, R32.1
- removed net N$14: JP6.23, JP6.24, JP7.23, R31.1
- removed net N$15: JP6.21, JP6.22, JP7.21, R30.1
- removed net N$16: JP6.19, JP6.20, JP7.19, R29.1
- removed net N$17: JP6.17, JP6.18, JP7.17, R28.1
- removed net N$18: JP6.15, JP6.16, JP7.15, R27.1
- removed net N$19: JP6.13, JP6.14, JP7.13, R25.1
- removed net N$20: JP6.11, JP6.12, JP7.11, R24.1
- removed net N$21: JP6.10, JP6.9, JP7.9, R23.1
- removed net N$23: JP6.5, JP6.6, JP7.5, R21.1
- removed net N$24: JP6.3, JP6.4, JP7.3, R20.1
- removed net N$25: JP10.1, JP10.2
- removed net N$26: JP6.1, JP6.2, JP7.1, R22.1
- removed net N$27: JP6.7, JP6.8, JP7.7, R33.1
- removed net N$28: JP6.27, JP6.28, JP7.27, R34.1
- removed net N$29: JP10.3, JP10.4
- removed net N$30: JP10.5, JP10.6
- removed net N$5: JP2.15, JP2.16, JP3.16, R14.1
- removed net N$6: JP2.13, JP2.14, JP3.14, R13.1
- removed net N$7: JP2.11, JP2.12, JP3.12, R10.1
- removed net N$8: JP2.10, JP2.9, JP3.10, R9.1
- removed net N$9: JP2.7, JP2.8, JP3.8, R8.1
- removed net USBDM: IC1.USBDM, X1.D-
- removed net USBDP: IC1.USBDP, X1.D+
- new net !RESET: !RESET.1, IC3.!RESET, R35.1
- new net !SHDN: JP36.2, R37.2, U2.!SHDN
- new net !SUSPEND: !SUSPEND.1, IC3.!SUSPEND
- new net 3V3_IN: C37.+, C4.1, D1.C, R37.1, U2.IN
- new net 5V_USB: D2.C, VUSB.1
- new net BTN0: B1.P$4, C6.2, JP38.1, R51.1
- new net BTN1: B2.P$4, C11.2, JP38.2, R50.1
- new net CHR0: CHR0.1, IC3.CHR0
- new net CHR1: CHR1.1, IC3.CHR1
- new net CHREN: CHREN.1, IC3.CHREN
- new net CLK/!RI: IC3.CLK/!RI, RI/CLK.1
- new net DCD: !DCD.1, IC3.!DCD
- new net DM: IC3.USBDM, USB.2, X1.D-
- new net DP: IC3.USBDP, USB.3, X1.D+
- new net DSR: !DSR.1, IC3.!DSR
- new net IO0_!RST!_: JP5.12, R31.2, T2.C, U1.IO0
- new net IO12_: JP1.11, R17.2, U1.IO12, U3.A2
- new net IO13_: JP1.12, R18.2, U1.IO13, U3.A0
- new net IO14_: JP1.10, R16.2, U1.IO14, U3.A1
- new net IO15_: JP5.14, R34.2, U1.IO15
- new net IO16_: JP5.10, R29.2, U1.IO16
- new net IO17_: JP5.9, R28.2, U1.IO17
- new net IO18_: JP5.7, R25.2, U1.IO18
- new net IO19_: JP5.6, R24.2, U1.IO19
- new net IO21_: JP5.5, R23.2, U1.IO21
- new net IO22_: JP5.2, R20.2, U1.IO22
- new net IO23_: JP5.1, R22.2, U1.IO23
- new net IO25_: JP1.7, R13.2, U1.IO25, U3.A5/SCL, U3.SCL
- new net IO26_: JP1.8, R14.2, U1.IO26, U3.A4/SDA, U3.SDA
- new net IO27_: JP1.9, R15.2, U1.IO27, U3.A3
- new net IO2_: JP5.13, R32.2, U1.IO2
- new net IO32_: JP1.5, R9.2, U1.IO32
- new net IO33_: JP1.6, R10.2, U1.IO33
- new net IO34_: JP1.3, R7.2, U1.IO34, U3.AREF
- new net IO35_: JP1.4, R8.2, U1.IO35
- new net IO4_: JP5.11, R30.2, U1.IO4
- new net IO5_: JP5.8, R27.2, U1.IO5
- new net LED0N: LED0N.C, R49.2
- new net LED0P: LED0P.A, R48.2
- new net LED1N: LED1N.C, R43.2
- new net LED1P: LED1P.A, R42.2
- new net LED2N: LED2N.C, R47.2
- new net LED2P: LED2P.A, R46.2
- new net LED3N: LED3N.C, R41.2
- new net LED3P: LED3P.A, R40.2
- new net LED4N: LED4N.C, R45.2
- new net LED4P: LED4P.A, R44.2
- new net LED5N: LED5N.C, R39.2
- new net LED5P: LED5P.A, R38.2
- new net LED_0: LEDS.6, R48.1, R49.1
- new net LED_1: LEDS.5, R42.1, R43.1
- new net LED_2: LEDS.4, R46.1, R47.1
- new net LED_3: LEDS.3, R40.1, R41.1
- new net LED_3V3_USB: LED_3V3_USB.C, R36.2
- new net LED_4: LEDS.2, R44.1, R45.1
- new net LED_5: LEDS.1, R38.1, R39.1
- new net N$32: SERVOS.3, SERVOS.4
- new net N$34: SERVOS.7, SERVOS.8
- new net N$36: SERVOS.11, SERVOS.12
- new net RX-LED: LED2.C, R2.1
- new net RXD0_: JP5.4, R11.2, R33.2, U1.RXD0
- new net RX_LED: IC3.RXLED/IO1, IO1/RXLED.1, R2.2
- new net SENSOR_VN_: JP1.2, R6.2, U1.SENSOR_VN
- new net SENSOR_VP_: JP1.1, R19.2, U1.SENSOR_VP
- new net SUSPEND: IC3.SUSPEND, R3.1, SUSPEND.1
- new net TX-LED: LED1.C, R1.1
- new net TXD0_: JP5.3, R12.2, R21.2, U1.TXD0
- new net TX_LED: IC3.TXLED/IO0, IO0/TXLED.1, R1.2
- new net USBID: USB.4, X1.ID
- new net USBIO3_RS485: IC3.RS485/IO2, IO2/RS485.1
- new net USBIO3_WAKEUP: IC3.WAKEUP/IO3, IO3/WAKEUP.1
- new net USBIO4: IC3.IO4, IO4.1
- new net USBIO5: IC3.IO5, IO5.1
- new net USBIO6: IC3.IO6, IO6.1
- new net VCCIO: C1.1, C2.1, IC3.VCC, LED1.A, LED2.A, LED3.A, LED_3V3_USB.A, R35.2, VCCIO.2, VCCIO.4, VCCIO.6
- new net VUSB: C3.1, C7.1, D2.A, IC3.VBUS, IC3.VREGIN, USB.1, X1.VBUS
- net !DTR: now also !DTR.1, IC3.!DTR; no longer IC1.!DTR
- net !RTS: now also !RTS.1, IC3.!RTS; no longer IC1.!RTS
- net +3V3: now also JP11.8, LED0N.A, LED1N.A, LED2N.A, LED3N.A, LED4N.A, LED5N.A, PWR_1.10, PWR_1.12, PWR_1.14, PWR_1.16, PWR_1.18, PWR_1.2, PWR_1.20, PWR_1.22, PWR_1.24, PWR_1.4, PWR_1.6, PWR_1.8, PWR_2.10, PWR_2.12, PWR_2.14, PWR_2.16, PWR_2.18, PWR_2.2, PWR_2.20, PWR_2.22, PWR_2.24, PWR_2.26, PWR_2.28, PWR_2.4, PWR_2.6, PWR_2.8, R50.2, R51.2, U3.3V, U3.IOREF; no longer C1.1, C6.2, IC1.VCCIO, LED0-N.A, LED1-N.A, LED2-N.A, LED3-N.A, LED_CBUS2.A, LED_CBUS3.A, LED_CBUS4.A, PWR_1.1, PWR_1.11, PWR_1.13, PWR_1.15, PWR_1.17, PWR_1.19, PWR_1.21, PWR_1.23, PWR_1.3, PWR_1.5, PWR_1.7, PWR_1.9, PWR_2.1, PWR_2.11, PWR_2.13, PWR_2.15, PWR_2.17, PWR_2.19, PWR_2.21, PWR_2.23, PWR_2.25, PWR_2.27, PWR_2.3, PWR_2.5, PWR_2.7, PWR_2.9
- net +5V: now also +5V.1, +5V.11, +5V.3, +5V.5, +5V.7, +5V.9, C10.1, C20.1, C67.1, C70.1, C8.1, C9.1, D1.A, PWR_1.1, PWR_1.11, PWR_1.13, PWR_1.15, PWR_1.17, PWR_1.19, PWR_1.21, PWR_1.23, PWR_1.3, PWR_1.5, PWR_1.7, PWR_1.9, PWR_2.1, PWR_2.11, PWR_2.13, PWR_2.15, PWR_2.17, PWR_2.19, PWR_2.21, PWR_2.23, PWR_2.25, PWR_2.27, PWR_2.3, PWR_2.5, PWR_2.7, PWR_2.9, U3.5V, VUSB.2; no longer C10.2, C11.2, C12.2, C8.+, C9.2, D1.C, D2.A, JP9.2, JP9.4, JP9.6, JP9.8, PWR_1.10, PWR_1.12, PWR_1.14, PWR_1.16, PWR_1.18, PWR_1.2, PWR_1.20, PWR_1.22, PWR_1.24, PWR_1.4, PWR_1.6, PWR_1.8, PWR_2.10, PWR_2.12, PWR_2.14, PWR_2.16, PWR_2.18, PWR_2.2, PWR_2.20, PWR_2.22, PWR_2.24, PWR_2.26, PWR_2.28, PWR_2.4, PWR_2.6, PWR_2.8
- net EN: now also EN.1, U3./RESET; no longer JP13.2
- net GND: now also +5V.10, +5V.12, +5V.2, +5V.4, +5V.6, +5V.8, B1.P$3, B2.P$3, C10.2, C20.2, C21.2, C37.-, C67.2, C70.2, C8.2, C9.2, EN.2, IC3.GND, JP11.7, JP36.1, LED0P.C, LED1P.C, LED2P.C, LED3P.C, LED4P.C, LED5P.C, R36.1, U3.GND, U3.GND1, U3.GND2, USB.5, VCC.1, VCC.3, VCC.5, VCCIO.1, VCCIO.3, VCCIO.5; no longer C10.1, C12.1, C13.2, C14.-, C8.-, C9.1, IC1.GND, IC1.GND@1, IC1.GND@2, IC1.GND@A, IC1.TEST, JP13.1, JP9.1, JP9.3, JP9.5, JP9.7, LED0-P.C, LED1-P.C, LED2-P.C, LED3-P.C
- net IO0_!RST: now also JP6.23, JP6.24, JP7.23, R31.1, U3.D6; no longer JP11.12, JP5.12, R31.2, T2.C, U1.IO0
- net IO12: now also JP2.21, JP2.22, JP3.22, R17.1; no longer JP1.11, JP12.11, R17.2, U1.IO12
- net IO13: now also JP2.23, JP2.24, JP3.24, R18.1; no longer JP1.12, JP12.12, R18.2, U1.IO13
- net IO14: now also JP2.19, JP2.20, JP3.20, R16.1; no longer JP1.10, JP12.10, R16.2, U1.IO14
- net IO15: now also JP6.27, JP6.28, JP7.27, R34.1, U3.D4; no longer JP11.14, JP5.14, R34.2, U1.IO15
- net IO16: now also JP6.19, JP6.20, JP7.19, R29.1, U3.D8; no longer JP11.10, JP5.10, R29.2, U1.IO16
- net IO17: now also JP6.17, JP6.18, JP7.17, R28.1, U3.D9; no longer JP11.9, JP5.9, R28.2, U1.IO17
- net IO18: now also JP6.13, JP6.14, JP7.13, R25.1, U3.D11; no longer JP11.7, JP5.7, R25.2, U1.IO18
- net IO19: now also JP6.11, JP6.12, JP7.11, R24.1, U3.D12; no longer JP11.6, JP5.6, R24.2, U1.IO19
- net IO2: now also JP6.25, JP6.26, JP7.25, R32.1, U3.D5; no longer JP11.13, JP5.13, R32.2, U1.IO2
- net IO21: now also JP6.10, JP6.9, JP7.9, R23.1, U3.D13; no longer JP11.5, JP5.5, R23.2, U1.IO21
- net IO22: now also JP6.3, JP6.4, JP7.3, R20.1, U3.D3; no longer JP11.2, JP5.2, R20.2, U1.IO22
- net IO23: now also JP6.1, JP6.2, JP7.1, R22.1, U3.D2; no longer JP11.1, JP5.1, R22.2, U1.IO23
- net IO25: now also JP2.13, JP2.14, JP3.14, R13.1; no longer JP1.7, JP12.7, R13.2, U1.IO25
- net IO26: now also JP2.15, JP2.16, JP3.16, R14.1; no longer JP1.8, JP12.8, R14.2, U1.IO26
- net IO27: now also JP2.17, JP2.18, JP3.18, R15.1; no longer JP1.9, JP12.9, R15.2, U1.IO27
- net IO32: now also JP2.10, JP2.9, JP3.10, R9.1; no longer JP1.5, JP12.5, R9.2, U1.IO32
- net IO33: now also JP2.11, JP2.12, JP3.12, R10.1; no longer JP1.6, JP12.6, R10.2, U1.IO33
- net IO34: now also JP2.5, JP2.6, JP3.6, R7.1; no longer JP1.3, JP12.3, R7.2, U1.IO34
- net IO35: now also JP2.7, JP2.8, JP3.8, R8.1; no longer JP1.4, JP12.4, R8.2, U1.IO35
- net IO4: now also JP6.21, JP6.22, JP7.21, R30.1, U3.D7; no longer JP11.11, JP5.11, R30.2, U1.IO4
- net IO5: now also JP6.15, JP6.16, JP7.15, R27.1, U3.D10; no longer JP11.8, JP5.8, R27.2, U1.IO5
- net N$1: now also NC28.NC, U3.RESERVED; no longer JP2.23, JP2.24, JP3.24, R18.1
- net N$2: now also !CTS.1, IC3.!CTS; no longer JP2.21, JP2.22, JP3.22, R17.1
- net N$3: now also U3.VIN; no longer JP2.19, JP2.20, JP3.20, R16.1
- net N$31: now also SERVOS.1, SERVOS.2; no longer JP10.7, JP10.8
- net N$33: now also SERVOS.5, SERVOS.6; no longer C3.1, C7.1, D1.A, IC1.VCC, X1.VBUS
- net N$35: now also SERVOS.10, SERVOS.9; no longer LED3.1, R44.1, R45.1
- net N$4: now also LED3.C, R3.2; no longer JP2.17, JP2.18, JP3.18, R15.1
- net NC-CS: now also JP11.3; no longer JP13.5
- net NC-HOLD: now also JP11.1; no longer JP13.3
- net NC-MISO: now also JP11.6; no longer JP13.8
- net NC-MOSI: now also JP11.5; no longer JP13.7
- net NC-SCK: now also JP11.4; no longer JP13.6
- net NC-WP: now also JP11.2; no longer JP13.4
- net RXD: now also IC3.RXD, RXD.1; no longer IC1.RXD
- net RXD0: now also JP6.7, JP6.8, JP7.7, R33.1, U3.D0; no longer JP11.4, JP5.4, R11.2, R33.2, U1.RXD0
- net SENSOR_VN: now also JP2.3, JP2.4, JP3.4, R6.1; no longer JP1.2, JP12.2, R6.2, U1.SENSOR_VN
- net SENSOR_VP: now also JP2.1, JP2.2, JP3.2, R19.1; no longer JP1.1, JP12.1, R19.2, U1.SENSOR_VP
- net TXD: now also IC3.TXD, TXD.1; no longer IC1.TXD
- net TXD0: now also JP6.5, JP6.6, JP7.5, R21.1, U3.D1; no longer JP11.3, JP5.3, R12.2, R21.2, U1.TXD0
- net VCC: now also D5.A, VCC.2, VCC.4, VCC.6; no longer D3.A
- net VCC->5V: now also C21.1, D5.C; no longer C13.1, D3.C
Other:
- note added: "v2.0"
- note removed: "v1.0"
- moved on the sheet: C1, C10, C11, C2, C3, C4, C5, C6, C7, C9, D2, IC2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

Commit message: updated silkscreen (and added bSilk)
Other:
- note added: "v2.1"
- note removed: "v2.0"
Changed lines of the file:
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@@
 <?xml version="1.0" encoding="utf-8"?>
 <!DOCTYPE eagle SYSTEM "eagle.dtd">
-<eagle version="8.1.0">
+<eagle version="7.2.0">
 <drawing>
 <settings>
@@
 <grid distance="0.1" unitdist="inch" unit="inch" style="lines" multiple="1" display="no" altdistance="0.01" altunitdist="inch" altunit="inch"/>
 <layers>
-<layer number="1" name="Top" color="4" fill="1" visible="yes" active="no"/>
-<layer number="2" name="Route2" color="1" fill="3" visible="yes" active="no"/>
-<layer number="3" name="Route3" color="4" fill="3" visible="yes" active="no"/>
-<layer number="4" name="Route4" color="1" fill="4" visible="yes" active="no"/>
-<layer number="5" name="Route5" color="4" fill="4" visible="yes" active="no"/>
-<layer number="6" name="Route6" color="1" fill="8" visible="yes" active="no"/>
-<layer number="7" name="Route7" color="4" fill="8" visible="yes" active="no"/>
-<layer number="8" name="Route8" color="1" fill="2" visible="yes" active="no"/>
-<layer number="9" name="Route9" color="4" fill="2" visible="yes" active="no"/>
-<layer number="10" name="Route10" color="1" fill="7" visible="yes" active="no"/>
-<layer number="11" name="Route11" color="4" fill="7" visible="yes" active="no"/>
-<layer number="12" name="Route12" color="1" fill="5" visible="yes" active="no"/>
-<layer number="13" name="Route13" color="4" fill="5" visible="yes" active="no"/>
-<layer number="14" name="Route14" color="1" fill="6" visible="yes" active="no"/>
-<layer number="15" name="Route15" color="4" fill="6" visible="yes" active="no"/>
-<layer number="16" name="Bottom" color="1" fill="1" visible="yes" active="no"/>
-<layer number="17" name="Pads" color="2" fill="1" visible="yes" active="no"/>
-<layer number="18" name="Vias" color="2" fill="1" visible="yes" active="no"/>
-<layer number="19" name="Unrouted" color="6" fill="1" visible="yes" active="no"/>
-<layer number="20" name="Dimension" color="15" fill="1" visible="yes" active="no"/>
-<layer number="21" name="tPlace" color="7" fill="1" visible="yes" active="no"/>
-<layer number="22" name="bPlace" color="7" fill="1" visible="yes" active="no"/>
-<layer number="23" name="tOrigins" color="15" fill="1" visible="yes" active="no"/>
-<layer number="24" name="bOrigins" color="15" fill="1" visible="yes" active="no"/>
-<layer number="25" name="tNames" color="7" fill="1" visible="yes" active="no"/>
-<layer number="26" name="bNames" color="7" fill="1" visible="yes" active="no"/>
-<layer number="27" name="tValues" color="7" fill="1" visible="yes" active="no"/>
-<layer number="28" name="bValues" color="7" fill="1" visible="yes" active="no"/>
+<layer number="1" name="Top" color="4" fill="1" visible="no" active="no"/>
+<layer number="2" name="Route2" color="1" fill="3" visible="no" active="no"/>
+<layer number="3" name="Route3" color="4" fill="3" visible="no" active="no"/>
+<layer number="4" name="Route4" color="1" fill="4" visible="no" active="no"/>
+<layer number="5" name="Route5" color="4" fill="4" visible="no" active="no"/>
+<layer number="6" name="Route6" color="1" fill="8" visible="no" active="no"/>
+<layer number="7" name="Route7" color="4" fill="8" visible="no" active="no"/>
+<layer number="8" name="Route8" color="1" fill="2" visible="no" active="no"/>
+<layer number="9" name="Route9" color="4" fill="2" visible="no" active="no"/>
+<layer number="10" name="Route10" color="1" fill="7" visible="no" active="no"/>
+<layer number="11" name="Route11" color="4" fill="7" visible="no" active="no"/>
+<layer number="12" name="Route12" color="1" fill="5" visible="no" active="no"/>
+<layer number="13" name="Route13" color="4" fill="5" visible="no" active="no"/>
+<layer number="14" name="Route14" color="1" fill="6" visible="no" active="no"/>
+<layer number="15" name="Route15" color="4" fill="6" visible="no" active="no"/>
+<layer number="16" name="Bottom" color="1" fill="1" visible="no" active="no"/>
+<layer number="17" name="Pads" color="2" fill="1" visible="no" active="no"/>
+<layer number="18" name="Vias" color="2" fill="1" visible="no" active="no"/>
+<layer number="19" name="Unrouted" color="6" fill="1" visible="no" active="no"/>
+<layer number="20" name="Dimension" color="15" fill="1" visible="no" active="no"/>
+<layer number="21" name="tPlace" color="7" fill="1" visible="no" active="no"/>
+<layer number="22" name="bPlace" color="7" fill="1" visible="no" active="no"/>
+<layer number="23" name="tOrigins" color="15" fill="1" visible="no" active="no"/>
+<layer number="24" name="bOrigins" color="15" fill="1" visible="no" active="no"/>
+<layer number="25" name="tNames" color="7" fill="1" visible="no" active="no"/>
+<layer number="26" name="bNames" color="7" fill="1" visible="no" active="no"/>
+<layer number="27" name="tValues" color="7" fill="1" visible="no" active="no"/>
+<layer number="28" name="bValues" color="7" fill="1" visible="no" active="no"/>
 <layer number="29" name="tStop" color="7" fill="3" visible="no" active="no"/>
 <layer number="30" name="bStop" color="7" fill="6" visible="no" active="no"/>
@@
 <layer number="35" name="tGlue" color="7" fill="4" visible="no" active="no"/>
 <layer number="36" name="bGlue" color="7" fill="5" visible="no" active="no"/>
-<layer number="37" name="tTest" color="7" fill="1" visible="yes" active="no"/>
-<layer number="38" name="bTest" color="7" fill="1" visible="yes" active="no"/>
+<layer number="37" name="tTest" color="7" fill="1" visible="no" active="no"/>
+<layer number="38" name="bTest" color="7" fill="1" visible="no" active="no"/>
 <layer number="39" name="tKeepout" color="4" fill="11" visible="no" active="no"/>
 <layer number="40" name="bKeepout" color="1" fill="11" visible="no" active="no"/>
@@
 <layer number="44" name="Drills" color="7" fill="1" visible="no" active="no"/>
 <layer number="45" name="Holes" color="7" fill="1" visible="no" active="no"/>
-<layer number="46" name="Milling" color="3" fill="1" visible="yes" active="no"/>
-<layer number="47" name="Measures" color="7" fill="1" visible="yes" active="no"/>
-<layer number="48" name="Document" color="7" fill="1" visible="yes" active="no"/>
-<layer number="49" name="Reference" color="7" fill="1" visible="yes" active="no"/>
-<layer number="50" name="dxf" color="7" fill="1" visible="yes" active="no"/>
-<layer number="51" name="tDocu" color="7" fill="1" visible="yes" active="no"/>
-<layer number="52" name="bDocu" color="7" fill="1" visible="yes" active="no"/>
-<layer number="53" name="tGND_GNDA" color="7" fill="9" visible="yes" active="no"/>
-<layer number="54" name="bGND_GNDA" color="1" fill="9" visible="yes" active="no"/>
-<layer number="55" name="tPotisk" color="7" fill="1" visible="yes" active="no"/>
-<layer number="56" name="wert" color="7" fill="1" visible="yes" active="no"/>
-<layer number="57" name="tCAD" color="7" fill="1" visible="yes" active="no"/>
-<layer number="58" name="bNC" color="7" fill="1" visible="yes" active="no"/>
-<layer number="59" name="tCarbon" color="7" fill="1" visible="yes" active="no"/>
-<layer number="60" name="bCarbon" color="7" fill="1" visible="yes" active="no"/>
-<layer number="61" name="stand" color="7" fill="1" visible="yes" active="no"/>
+<layer number="46" name="Milling" color="3" fill="1" visible="no" active="no"/>
+<layer number="47" name="Measures" color="7" fill="1" visible="no" active="no"/>
+<layer number="48" name="Document" color="7" fill="1" visible="no" active="no"/>
+<layer number="49" name="Reference" color="7" fill="1" visible="no" active="no"/>
+<layer number="50" name="dxf" color="7" fill="1" visible="no" active="no"/>
+<layer number="51" name="tDocu" color="7" fill="1" visible="no" active="no"/>
+<layer number="52" name="bDocu" color="7" fill="1" visible="no" active="no"/>
+<layer number="53" name="tGND_GNDA" color="7" fill="9" visible="no" active="no"/>
+<layer number="54" name="bGND_GNDA" color="1" fill="9" visible="no" active="no"/>
+<layer number="55" name="tPotisk" color="7" fill="1" visible="no" active="no"/>
+<layer number="56" name="wert" color="7" fill="1" visible="no" active="no"/>
+<layer number="57" name="tCAD" color="7" fill="1" visible="no" active="no"/>
+<layer number="58" name="bNC" color="7" fill="1" visible="no" active="no"/>
+<layer number="59" name="tCarbon" color="7" fill="1" visible="no" active="no"/>
+<layer number="60" name="bCarbon" color="7" fill="1" visible="no" active="no"/>
+<layer number="61" name="stand" color="7" fill="1" visible="no" active="no"/>
 <layer number="90" name="Modules" color="5" fill="1" visible="no" active="yes"/>
 <layer number="91" name="Nets" color="2" fill="1" visible="yes" active="yes"/>
@@
 CC BY-SA 4.0</text>
 <text x="344.17" y="20.32" size="2.54" layer="97" font="vector" ratio="14">RobotikaBrno</text>
-<text x="374.65" y="5.08" size="2.54" layer="97" font="vector" ratio="14">v2.0</text>
+<text x="374.65" y="5.08" size="2.54" layer="97" font="vector" ratio="14">v2.1</text>
 <rectangle x1="338.570040625" y1="18.3900375" x2="338.783396875" y2="18.4002" layer="102"/>
 <rectangle x1="338.4278" y1="18.4002" x2="338.9256375" y2="18.41035625" layer="102"/>
