File: hardware/RB3200-ESP32universal.brd (EAGLE design)
At the start: 83.8 x 52.1 mm, 138 parts, among them IC2 7805, IC3 CP2102N-28, T1 BC337, T2 BC337, U1 ESP-WROOM-32, U2 UM18533, U3 ARDUINOR3-BPLACE, X1 USB-MICRO-B-BOTTOM

Commit message: Add enable pullup
This solves board flashing issues.
Parts:
- added C12: 1n/50V, rcl_upravena:C0603
- added R52: 12k, rcl_upravena:R0603
Connections:
- net +3V3: now also R52.2
- net EN: now also C12.1, R52.1
- net GND: now also C12.2
Routing:
- net EN: track 103.3 -> 105.0 mm
Changed lines of the file:
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@@
 <?xml version="1.0" encoding="utf-8"?>
 <!DOCTYPE eagle SYSTEM "eagle.dtd">
-<eagle version="7.2.0">
+<eagle version="7.7.0">
 <drawing>
 <settings>
@@
 <setting verticaltext="up"/>
 </settings>
-<grid distance="0.05" unitdist="inch" unit="mm" style="lines" multiple="2" display="yes" altdistance="0.3125" altunitdist="mm" altunit="mm"/>
+<grid distance="0.05" unitdist="inch" unit="mm" style="lines" multiple="1" display="yes" altdistance="0.3125" altunitdist="mm" altunit="mm"/>
 <layers>
-<layer number="1" name="Top" color="4" fill="1" visible="no" active="yes"/>
+<layer number="1" name="Top" color="4" fill="1" visible="yes" active="yes"/>
 <layer number="2" name="Route2" color="1" fill="3" visible="no" active="no"/>
 <layer number="3" name="Route3" color="4" fill="3" visible="no" active="no"/>
@@
 <layer number="14" name="Route14" color="1" fill="6" visible="no" active="no"/>
 <layer number="15" name="Route15" color="4" fill="6" visible="no" active="no"/>
-<layer number="16" name="Bottom" color="1" fill="1" visible="no" active="yes"/>
-<layer number="17" name="Pads" color="2" fill="1" visible="no" active="yes"/>
-<layer number="18" name="Vias" color="2" fill="1" visible="no" active="yes"/>
-<layer number="19" name="Unrouted" color="6" fill="1" visible="no" active="yes"/>
+<layer number="16" name="Bottom" color="1" fill="1" visible="yes" active="yes"/>
+<layer number="17" name="Pads" color="2" fill="1" visible="yes" active="yes"/>
+<layer number="18" name="Vias" color="2" fill="1" visible="yes" active="yes"/>
+<layer number="19" name="Unrouted" color="6" fill="1" visible="yes" active="yes"/>
 <layer number="20" name="Dimension" color="15" fill="1" visible="yes" active="yes"/>
 <layer number="21" name="tPlace" color="7" fill="1" visible="yes" active="yes"/>
-<layer number="22" name="bPlace" color="7" fill="1" visible="no" active="yes"/>
-<layer number="23" name="tOrigins" color="15" fill="1" visible="no" active="yes"/>
-<layer number="24" name="bOrigins" color="15" fill="1" visible="no" active="yes"/>
-<layer number="25" name="tNames" color="7" fill="1" visible="no" active="yes"/>
-<layer number="26" name="bNames" color="7" fill="1" visible="no" active="yes"/>
-<layer number="27" name="tValues" color="7" fill="1" visible="no" active="yes"/>
-<layer number="28" name="bValues" color="7" fill="1" visible="no" active="yes"/>
+<layer number="22" name="bPlace" color="7" fill="1" visible="yes" active="yes"/>
+<layer number="23" name="tOrigins" color="15" fill="1" visible="yes" active="yes"/>
+<layer number="24" name="bOrigins" color="15" fill="1" visible="yes" active="yes"/>
+<layer number="25" name="tNames" color="7" fill="1" visible="yes" active="yes"/>
+<layer number="26" name="bNames" color="7" fill="1" visible="yes" active="yes"/>
+<layer number="27" name="tValues" color="7" fill="1" visible="yes" active="yes"/>
+<layer number="28" name="bValues" color="7" fill="1" visible="yes" active="yes"/>
 <layer number="29" name="tStop" color="7" fill="3" visible="no" active="yes"/>
 <layer number="30" name="bStop" color="7" fill="6" visible="no" active="yes"/>
@@
 <layer number="47" name="Measures" color="7" fill="1" visible="no" active="yes"/>
 <layer number="48" name="Document" color="7" fill="1" visible="no" active="yes"/>
-<layer number="49" name="Reference" color="7" fill="1" visible="no" active="yes"/>
+<layer number="49" name="Reference" color="7" fill="1" visible="yes" active="yes"/>
 <layer number="50" name="dxf" color="7" fill="1" visible="no" active="no"/>
-<layer number="51" name="tDocu" color="7" fill="1" visible="no" active="yes"/>
-<layer number="52" name="bDocu" color="7" fill="1" visible="no" active="yes"/>
+<layer number="51" name="tDocu" color="7" fill="1" visible="yes" active="yes"/>
+<layer number="52" name="bDocu" color="7" fill="1" visible="yes" active="yes"/>
 <layer number="53" name="tGND_GNDA" color="7" fill="9" visible="no" active="no"/>
 <layer number="54" name="bGND_GNDA" color="1" fill="9" visible="no" active="no"/>
@@
 <element name="R50" library="rcl_upravena" package="R0603" value="10k" x="66.04" y="7.62" rot="R90"/>
 <element name="R51" library="rcl_upravena" package="R0603" value="10k" x="67.31" y="7.62" rot="R90"/>
+<element name="R52" library="rcl_upravena" package="R0603" value="12k" x="53.6525" y="9.8475" rot="R270"/>
+<element name="C12" library="rcl_upravena" package="C0603" value="1n/50V" x="52.72" y="12.6175" rot="MR90"/>
 </elements>
 <signals>
@@
 <via x="54.9275" y="8.89" extent="1-16" drill="0.6"/>
 <wire x1="54.9275" y1="8.89" x2="56.8325" y2="10.795" width="0.8128" layer="16"/>
-<wire x1="51.16" y1="8.875" x2="54.9125" y2="8.875" width="0.8128" layer="1"/>
+<wire x1="51.16" y1="8.875" x2="53.34" y2="8.875" width="0.8128" layer="1"/>
+<wire x1="53.34" y1="8.875" x2="54.9125" y2="8.875" width="0.8128" layer="1"/>
 <wire x1="54.9125" y1="8.875" x2="54.9275" y2="8.89" width="0.8128" layer="1"/>
 <wire x1="66.04" y1="19.05" x2="78.74" y2="19.05" width="0.8128" layer="16"/>
@@
 <wire x1="67.31" y1="12.7" x2="66.04" y2="13.97" width="0.4064" layer="1"/>
 <wire x1="66.04" y1="8.47" x2="67.31" y2="8.47" width="0.4064" layer="1"/>
+<contactref element="R52" pad="2"/>
+<wire x1="53.6525" y1="8.9975" x2="53.4625" y2="8.9975" width="0.4064" layer="1"/>
+<wire x1="53.4625" y1="8.9975" x2="53.34" y2="8.875" width="0.4064" layer="1"/>
 </signal>
 <signal name="GND">
@@
 <wire x1="59.3725" y1="41.43375" x2="59.74625" y2="41.8075" width="0.6096" layer="16"/>
 <wire x1="59.74625" y1="41.8075" x2="59.74625" y2="42.545" width="0.6096" layer="16"/>
-<wire x1="59.3725" y1="40.48125" x2="59.3725" y2="39.21125" width="0.6096" layer="16"/>
-<wire x1="59.3725" y1="39.21125" x2="59.3725" y2="37.1475" width="0.6096" layer="16"/>
+<wire x1="59.3725" y1="40.48125" x2="59.3725" y2="37.1475" width="0.6096" layer="16"/>
 <wire x1="59.3725" y1="37.1475" x2="59.74625" y2="36.77375" width="0.6096" layer="16"/>
 <wire x1="59.74625" y1="36.77375" x2="59.74625" y2="36.03625" width="0.6096" layer="16"/>
@@
 <wire x1="42.21" y1="15.305" x2="42.21" y2="19.0325" width="0.8128" layer="1"/>
 <wire x1="42.21" y1="19.0325" x2="47.61" y2="24.4325" width="0.8128" layer="1"/>
+<contactref element="C12" pad="2"/>
 </signal>
 <signal name="TXD">
@@
 <wire x1="55.88" y1="5.08" x2="57.15" y2="3.81" width="0.4064" layer="1"/>
 <wire x1="55.88" y1="9.495" x2="55.88" y2="5.08" width="0.4064" layer="1"/>
-<wire x1="64.77" y1="7.62" x2="64.77" y2="15.24" width="0.4064" layer="1"/>
+<wire x1="64.77" y1="5.23875" x2="64.77" y2="15.24" width="0.4064" layer="1"/>
 <via x="52.54625" y="10.795" extent="1-16" drill="0.3"/>
 <wire x1="52.54625" y1="10.795" x2="52.22875" y2="10.4775" width="0.4064" layer="16"/>
@@
 <wire x1="51.16" y1="10.145" x2="52.54625" y2="10.145" width="0.4064" layer="1"/>
 <wire x1="52.54625" y1="10.145" x2="52.54625" y2="10.795" width="0.4064" layer="1"/>
-<wire x1="52.54625" y1="10.145" x2="55.23" y2="10.145" width="0.4064" layer="1"/>
+<wire x1="52.54625" y1="10.145" x2="53.34" y2="10.145" width="0.4064" layer="1"/>
+<wire x1="53.34" y1="10.145" x2="55.23" y2="10.145" width="0.4064" layer="1"/>
 <wire x1="52.07" y1="31.75" x2="52.07" y2="29.845" width="0.254" layer="16"/>
 <wire x1="52.07" y1="29.845" x2="50.165" y2="27.94" width="0.254" layer="16"/>
@@
 <wire x1="35.56" y1="29.845" x2="34.925" y2="30.48" width="0.254" layer="16"/>
 <wire x1="34.925" y1="30.48" x2="31.115" y2="30.48" width="0.254" layer="16"/>
-<wire x1="31.115" y1="30.48" x2="30.48" y2="29.845" width="0.254" layer="16"/>
-<wire x1="30.48" y1="29.845" x2="29.68625" y2="29.05125" width="0.254" layer="16"/>
+<wire x1="31.115" y1="30.48" x2="29.68625" y2="29.05125" width="0.254" layer="16"/>
 <wire x1="29.68625" y1="29.05125" x2="29.0625" y2="29.05125" width="0.254" layer="16"/>
 <wire x1="29.0625" y1="29.05125" x2="29.05125" y2="29.0625" width="0.254" layer="16"/>
 <wire x1="57.15" y1="3.81" x2="63.34125" y2="3.81" width="0.4064" layer="1"/>
 <wire x1="63.34125" y1="3.81" x2="64.77" y2="5.23875" width="0.4064" layer="1"/>
-<wire x1="64.77" y1="5.23875" x2="64.77" y2="7.62" width="0.4064" layer="1"/>
+<contactref element="C12" pad="1"/>
+<contactref element="R52" pad="1"/>
+<wire x1="53.6525" y1="10.6975" x2="53.6525" y2="10.4575" width="0.4064" layer="1"/>
+<wire x1="53.6525" y1="10.4575" x2="53.34" y2="10.145" width="0.4064" layer="1"/>
+<wire x1="52.54625" y1="10.795" x2="52.72" y2="10.96875" width="0.4064" layer="16" curve="90"/>
+<wire x1="52.72" y1="10.96875" x2="52.72" y2="11.7675" width="0.4064" layer="16"/>
 </signal>
 <signal name="NC-HOLD">

Commit message: Change EN pullup value to simplify BOM
Parts:
- R52: value 12k -> 10k
Changed lines of the file:
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@@
 <element name="R50" library="rcl_upravena" package="R0603" value="10k" x="66.04" y="7.62" rot="R90"/>
 <element name="R51" library="rcl_upravena" package="R0603" value="10k" x="67.31" y="7.62" rot="R90"/>
-<element name="R52" library="rcl_upravena" package="R0603" value="12k" x="53.6525" y="9.8475" rot="R270"/>
+<element name="R52" library="rcl_upravena" package="R0603" value="10k" x="53.6525" y="9.8475" rot="R270"/>
 <element name="C12" library="rcl_upravena" package="C0603" value="1n/50V" x="52.72" y="12.6175" rot="MR90"/>
 </elements>
